File: OkGo 2/ignition/ignition.sch (KiCad schematic (older format))
At the start: 40 parts, among them P101 JST_XH_F, P102 JST_XH_M, P103 CHARGE_CASE, P104 BATT, P105 BATT, P106 SMA, SW101 20A ROCKER, U101 CLIP, U102 FUSE 15A, U103 SWD, U104 BEZEL, U105 RFM95W, U106 STM32F071CBT6, U107 TSR 0.5-2433, Y101 8MHz

Commit message: minor schematic changes
Parts:
- added P107: ARM_LED, common:JST-PA-2, symbol CONN_01X02
- added P108: ARM_LED, symbol CONN_01X02
Connections:
- net DISARM_LED: now also P107.1 (P1); no longer D102.2 (A)
- net at R103.1: now also P107.2 (P2); no longer D102.1 (K)
- new net: D102.1 (K), P108.2 (P2)
- new net: D102.2 (A), P108.1 (P1)
Other:
- note added: "11.1V 5.8Ah"
- note removed: "3.7V 5.8Ah"
- moved on the sheet: R103
Changed lines of the file:
@@
 $EndDescr
 $Comp
-L PWR_FLAG #FLG01
+L PWR_FLAG #FLG101
 U 1 1 5562BA6E
 P 4900 1200
-F 0 "#FLG01" H 4900 1295 50  0001 C CNN
+F 0 "#FLG101" H 4900 1295 50  0001 C CNN
 F 1 "PWR_FLAG" H 4900 1380 50  0000 C CNN
 F 2 "" H 4900 1200 60  0000 C CNN
@@
 $EndComp
 $Comp
-L PWR_FLAG #FLG02
+L PWR_FLAG #FLG102
 U 1 1 5562BA86
 P 4900 1400
-F 0 "#FLG02" H 4900 1495 50  0001 C CNN
+F 0 "#FLG102" H 4900 1495 50  0001 C CNN
 F 1 "PWR_FLAG" H 4900 1580 50  0000 C CNN
 F 2 "" H 4900 1400 60  0000 C CNN
@@
 $EndComp
 $Comp
-L GND #PWR03
+L GND #PWR105
 U 1 1 5562BBD7
 P 5625 2050
-F 0 "#PWR03" H 5625 1800 50  0001 C CNN
+F 0 "#PWR105" H 5625 1800 50  0001 C CNN
 F 1 "GND" H 5625 1900 50  0000 C CNN
 F 2 "" H 5625 2050 60  0000 C CNN
@@
 $EndComp
 $Comp
-L GND #PWR04
+L GND #PWR117
 U 1 1 5562BDA6
 P 6050 6850
-F 0 "#PWR04" H 6050 6600 50  0001 C CNN
+F 0 "#PWR117" H 6050 6600 50  0001 C CNN
 F 1 "GND" H 6050 6700 50  0000 C CNN
 F 2 "" H 6050 6850 60  0000 C CNN
@@
 $EndComp
 $Comp
-L +3V3 #PWR05
+L +3V3 #PWR114
 U 1 1 5562C50D
 P 6650 6250
-F 0 "#PWR05" H 6650 6100 50  0001 C CNN
+F 0 "#PWR114" H 6650 6100 50  0001 C CNN
 F 1 "+3V3" H 6650 6390 50  0000 C CNN
 F 2 "" H 6650 6250 60  0000 C CNN
@@
 $EndComp
 $Comp
-L +3V3 #PWR06
+L +3V3 #PWR101
 U 1 1 5562CAD0
 P 9250 1100
-F 0 "#PWR06" H 9250 950 50  0001 C CNN
+F 0 "#PWR101" H 9250 950 50  0001 C CNN
 F 1 "+3V3" H 9250 1240 50  0000 C CNN
 F 2 "" H 9250 1100 60  0000 C CNN
@@
 $EndComp
 $Comp
-L GND #PWR07
+L GND #PWR104
 U 1 1 5562CB22
 P 9250 1600
-F 0 "#PWR07" H 9250 1350 50  0001 C CNN
+F 0 "#PWR104" H 9250 1350 50  0001 C CNN
 F 1 "GND" H 9250 1450 50  0000 C CNN
 F 2 "" H 9250 1600 60  0000 C CNN
@@
 NoConn ~ 10550 1450
 $Comp
-L +3V3 #PWR08
+L +3V3 #PWR109
 U 1 1 5562D38F
 P 8600 4875
-F 0 "#PWR08" H 8600 4725 50  0001 C CNN
+F 0 "#PWR109" H 8600 4725 50  0001 C CNN
 F 1 "+3V3" H 8600 5015 50  0000 C CNN
 F 2 "" H 8600 4875 60  0000 C CNN
@@
 $EndComp
 $Comp
-L GND #PWR09
+L GND #PWR110
 U 1 1 5562D3AE
 P 8300 5350
-F 0 "#PWR09" H 8300 5100 50  0001 C CNN
+F 0 "#PWR110" H 8300 5100 50  0001 C CNN
 F 1 "GND" H 8300 5200 50  0000 C CNN
 F 2 "" H 8300 5350 60  0000 C CNN
@@
 $EndComp
 $Comp
-L GND #PWR010
+L GND #PWR115
 U 1 1 5562DF61
 P 10275 6300
-F 0 "#PWR010" H 10275 6050 50  0001 C CNN
+F 0 "#PWR115" H 10275 6050 50  0001 C CNN
 F 1 "GND" H 10275 6150 50  0000 C CNN
 F 2 "" H 10275 6300 60  0000 C CNN
@@
 $EndComp
 $Comp
-L +3V3 #PWR011
+L +3V3 #PWR106
 U 1 1 5562E586
 P 1450 3950
-F 0 "#PWR011" H 1450 3800 50  0001 C CNN
+F 0 "#PWR106" H 1450 3800 50  0001 C CNN
 F 1 "+3V3" H 1450 4090 50  0000 C CNN
 F 2 "" H 1450 3950 60  0000 C CNN
@@
 $EndComp
 $Comp
-L GND #PWR012
+L GND #PWR111
 U 1 1 5562F2E9
 P 1500 5500
-F 0 "#PWR012" H 1500 5250 50  0001 C CNN
+F 0 "#PWR111" H 1500 5250 50  0001 C CNN
 F 1 "GND" H 1500 5350 50  0000 C CNN
 F 2 "" H 1500 5500 60  0000 C CNN
@@
 $EndComp
 $Comp
-L GND #PWR013
+L GND #PWR108
 U 1 1 5562F9AC
 P 3950 4700
-F 0 "#PWR013" H 3950 4450 50  0001 C CNN
+F 0 "#PWR108" H 3950 4450 50  0001 C CNN
 F 1 "GND" H 3950 4550 50  0000 C CNN
 F 2 "" H 3950 4700 60  0000 C CNN
@@
 $EndComp
 $Comp
-L GND #PWR014
+L GND #PWR113
 U 1 1 5563121C
 P 4750 5950
-F 0 "#PWR014" H 4750 5700 50  0001 C CNN
+F 0 "#PWR113" H 4750 5700 50  0001 C CNN
 F 1 "GND" H 4750 5800 50  0000 C CNN
 F 2 "" H 4750 5950 60  0000 C CNN
@@
 Bat: 3*4.2V\nMon: 3.1V
 $Comp
-L +3V3 #PWR015
+L +3V3 #PWR107
 U 1 1 559CAD6D
 P 1900 4500
-F 0 "#PWR015" H 1900 4350 50  0001 C CNN
+F 0 "#PWR107" H 1900 4350 50  0001 C CNN
 F 1 "+3V3" H 1900 4640 50  0000 C CNN
 F 2 "" H 1900 4500 60  0000 C CNN
@@
 $EndComp
 $Comp
-L GND #PWR016
+L GND #PWR112
 U 1 1 559E749A
 P 10375 5850
-F 0 "#PWR016" H 10375 5600 50  0001 C CNN
+F 0 "#PWR112" H 10375 5600 50  0001 C CNN
 F 1 "GND" H 10375 5700 50  0001 C CNN
 F 2 "" H 10375 5850 60  0000 C CNN
@@
 $EndComp
 $Comp
-L GND #PWR017
+L GND #PWR103
 U 1 1 55A1A3D6
 P 5425 1400
-F 0 "#PWR017" H 5425 1150 50  0001 C CNN
+F 0 "#PWR103" H 5425 1150 50  0001 C CNN
 F 1 "GND" H 5425 1250 50  0000 C CNN
 F 2 "" H 5425 1400 60  0000 C CNN
@@
 $EndComp
 $Comp
-L +BATT #PWR018
+L +BATT #PWR102
 U 1 1 55A1ACA2
 P 5425 1200
-F 0 "#PWR018" H 5425 1050 50  0001 C CNN
+F 0 "#PWR102" H 5425 1050 50  0001 C CNN
 F 1 "+BATT" H 5425 1340 50  0000 C CNN
 F 2 "" H 5425 1200 60  0000 C CNN
@@
 $EndComp
 $Comp
-L +BATT #PWR019
+L +BATT #PWR116
 U 1 1 55A85387
 P 5550 6400
-F 0 "#PWR019" H 5550 6250 50  0001 C CNN
+F 0 "#PWR116" H 5550 6250 50  0001 C CNN
 F 1 "+BATT" H 5550 6540 50  0000 C CNN
 F 2 "" H 5550 6400 60  0000 C CNN
@@
 L R R103
 U 1 1 55A8E9D5
-P 3050 2700
-F 0 "R103" V 3130 2700 50  0000 C CNN
-F 1 "75R" V 3050 2700 50  0000 C CNN
-F 2 "Resistors_SMD:R_0805" V 2980 2700 30  0001 C CNN
-F 3 "" H 3050 2700 30  0000 C CNN
-F 4 "2331781" H 3050 2700 60  0001 C CNN "Farnell"
-	1    3050 2700
+P 2225 2700
+F 0 "R103" V 2305 2700 50  0000 C CNN
+F 1 "75R" V 2225 2700 50  0000 C CNN
+F 2 "Resistors_SMD:R_0805" V 2155 2700 30  0001 C CNN
+F 3 "" H 2225 2700 30  0000 C CNN
+F 4 "2331781" H 2225 2700 60  0001 C CNN "Farnell"
+	1    2225 2700
 	0    1    1    0
 $EndComp
-Text Label 2900 2700 2    60   ~ 0
+Text Label 2075 2700 2    60   ~ 0
 ARM_LED
-Text Label 2900 2900 2    60   ~ 0
+Text Label 2075 2900 2    60   ~ 0
 DISARM_LED
 Text Label 5900 2850 0    60   ~ 0
@@
 	1    0    0    -1
 $EndComp
-Text Notes 2450 2600 0    60   ~ 0
+Text Notes 1625 2600 0    60   ~ 0
 RED: 1.95V 20mA
-Text Notes 2400 3025 0    60   ~ 0
+Text Notes 1575 3025 0    60   ~ 0
 GREEN: 2.1V 20mA
 $Comp
@@
 Wire Wire Line
 	3825 1250 3775 1250
-Text Notes 750  1225 0    60   ~ 0
-3.7V 5.8Ah
+Text Notes 700  1225 0    60   ~ 0
+11.1V 5.8Ah
 $Comp
 L CONN_01X04 P102
@@
 	1    0    0    -1
 $EndComp
-Wire Wire Line
-	2900 2900 3600 2900
-Wire Wire Line
-	3200 2700 3300 2700
 Wire Wire Line
 	3600 2900 3600 2700
@@
 	6650 6400 6650 6250
 Connection ~ 6650 6400
+$Comp
+L CONN_01X02 P107
+U 1 1 55C63A4F
+P 2750 2750
+F 0 "P107" H 2725 2600 50  0000 C CNN
+F 1 "ARM_LED" H 2650 2900 50  0000 C CNN
+F 2 "common:JST-PA-2" H 2750 2750 60  0001 C CNN
+F 3 "" H 2750 2750 60  0000 C CNN
+F 4 "1830747" H 2750 2750 60  0001 C CNN "Farnell"
+	1    2750 2750
+	1    0    0    1
+$EndComp
+$Comp
+L CONN_01X02 P108
+U 1 1 55C63A57
+P 2900 2750
+F 0 "P108" H 2850 2600 50  0000 C CNN
+F 1 "ARM_LED" H 2800 2900 50  0000 C CNN
+F 2 "" H 2900 2750 60  0001 C CNN
+F 3 "" H 2900 2750 60  0000 C CNN
+F 4 "1830726" H 2900 2750 60  0001 C CNN "Farnell"
+	1    2900 2750
+	-1   0    0    1
+$EndComp
+Wire Wire Line
+	2375 2700 2550 2700
+Wire Wire Line
+	2075 2900 2400 2900
+Wire Wire Line
+	2400 2900 2400 2800
+Wire Wire Line
+	2400 2800 2550 2800
+Wire Wire Line
+	3100 2700 3300 2700
+Wire Wire Line
+	3100 2800 3300 2800
+Wire Wire Line
+	3300 2800 3300 2900
+Wire Wire Line
+	3300 2900 3600 2900
 $EndSCHEMATC

Commit message: ignition; first attempt at placement
Parts:
- P107: footprint common:JST-PA-2 -> ignition:JST-PA-2-VERT; Farnell 1830747 -> 1830734
Changed lines of the file:
@@
 $EndDescr
 $Comp
-L PWR_FLAG #FLG101
+L PWR_FLAG #FLG01
 U 1 1 5562BA6E
 P 4900 1200
-F 0 "#FLG101" H 4900 1295 50  0001 C CNN
+F 0 "#FLG01" H 4900 1295 50  0001 C CNN
 F 1 "PWR_FLAG" H 4900 1380 50  0000 C CNN
 F 2 "" H 4900 1200 60  0000 C CNN
@@
 $EndComp
 $Comp
-L PWR_FLAG #FLG102
+L PWR_FLAG #FLG02
 U 1 1 5562BA86
 P 4900 1400
-F 0 "#FLG102" H 4900 1495 50  0001 C CNN
+F 0 "#FLG02" H 4900 1495 50  0001 C CNN
 F 1 "PWR_FLAG" H 4900 1580 50  0000 C CNN
 F 2 "" H 4900 1400 60  0000 C CNN
@@
 $EndComp
 $Comp
-L GND #PWR105
+L GND #PWR03
 U 1 1 5562BBD7
 P 5625 2050
-F 0 "#PWR105" H 5625 1800 50  0001 C CNN
+F 0 "#PWR03" H 5625 1800 50  0001 C CNN
 F 1 "GND" H 5625 1900 50  0000 C CNN
 F 2 "" H 5625 2050 60  0000 C CNN
@@
 $EndComp
 $Comp
-L GND #PWR117
+L GND #PWR04
 U 1 1 5562BDA6
 P 6050 6850
-F 0 "#PWR117" H 6050 6600 50  0001 C CNN
+F 0 "#PWR04" H 6050 6600 50  0001 C CNN
 F 1 "GND" H 6050 6700 50  0000 C CNN
 F 2 "" H 6050 6850 60  0000 C CNN
@@
 $EndComp
 $Comp
-L +3V3 #PWR114
+L +3V3 #PWR05
 U 1 1 5562C50D
 P 6650 6250
-F 0 "#PWR114" H 6650 6100 50  0001 C CNN
+F 0 "#PWR05" H 6650 6100 50  0001 C CNN
 F 1 "+3V3" H 6650 6390 50  0000 C CNN
 F 2 "" H 6650 6250 60  0000 C CNN
@@
 $EndComp
 $Comp
-L +3V3 #PWR101
+L +3V3 #PWR06
 U 1 1 5562CAD0
 P 9250 1100
-F 0 "#PWR101" H 9250 950 50  0001 C CNN
+F 0 "#PWR06" H 9250 950 50  0001 C CNN
 F 1 "+3V3" H 9250 1240 50  0000 C CNN
 F 2 "" H 9250 1100 60  0000 C CNN
@@
 $EndComp
 $Comp
-L GND #PWR104
+L GND #PWR07
 U 1 1 5562CB22
 P 9250 1600
-F 0 "#PWR104" H 9250 1350 50  0001 C CNN
+F 0 "#PWR07" H 9250 1350 50  0001 C CNN
 F 1 "GND" H 9250 1450 50  0000 C CNN
 F 2 "" H 9250 1600 60  0000 C CNN
@@
 NoConn ~ 10550 1450
 $Comp
-L +3V3 #PWR109
+L +3V3 #PWR08
 U 1 1 5562D38F
 P 8600 4875
-F 0 "#PWR109" H 8600 4725 50  0001 C CNN
+F 0 "#PWR08" H 8600 4725 50  0001 C CNN
 F 1 "+3V3" H 8600 5015 50  0000 C CNN
 F 2 "" H 8600 4875 60  0000 C CNN
@@
 $EndComp
 $Comp
-L GND #PWR110
+L GND #PWR09
 U 1 1 5562D3AE
 P 8300 5350
-F 0 "#PWR110" H 8300 5100 50  0001 C CNN
+F 0 "#PWR09" H 8300 5100 50  0001 C CNN
 F 1 "GND" H 8300 5200 50  0000 C CNN
 F 2 "" H 8300 5350 60  0000 C CNN
@@
 $EndComp
 $Comp
-L GND #PWR115
+L GND #PWR010
 U 1 1 5562DF61
 P 10275 6300
-F 0 "#PWR115" H 10275 6050 50  0001 C CNN
+F 0 "#PWR010" H 10275 6050 50  0001 C CNN
 F 1 "GND" H 10275 6150 50  0000 C CNN
 F 2 "" H 10275 6300 60  0000 C CNN
@@
 $EndComp
 $Comp
-L +3V3 #PWR106
+L +3V3 #PWR011
 U 1 1 5562E586
 P 1450 3950
-F 0 "#PWR106" H 1450 3800 50  0001 C CNN
+F 0 "#PWR011" H 1450 3800 50  0001 C CNN
 F 1 "+3V3" H 1450 4090 50  0000 C CNN
 F 2 "" H 1450 3950 60  0000 C CNN
@@
 $EndComp
 $Comp
-L GND #PWR111
+L GND #PWR012
 U 1 1 5562F2E9
 P 1500 5500
-F 0 "#PWR111" H 1500 5250 50  0001 C CNN
+F 0 "#PWR012" H 1500 5250 50  0001 C CNN
 F 1 "GND" H 1500 5350 50  0000 C CNN
 F 2 "" H 1500 5500 60  0000 C CNN
@@
 $EndComp
 $Comp
-L GND #PWR108
+L GND #PWR013
 U 1 1 5562F9AC
 P 3950 4700
-F 0 "#PWR108" H 3950 4450 50  0001 C CNN
+F 0 "#PWR013" H 3950 4450 50  0001 C CNN
 F 1 "GND" H 3950 4550 50  0000 C CNN
 F 2 "" H 3950 4700 60  0000 C CNN
@@
 $EndComp
 $Comp
-L GND #PWR113
+L GND #PWR014
 U 1 1 5563121C
 P 4750 5950
-F 0 "#PWR113" H 4750 5700 50  0001 C CNN
+F 0 "#PWR014" H 4750 5700 50  0001 C CNN
 F 1 "GND" H 4750 5800 50  0000 C CNN
 F 2 "" H 4750 5950 60  0000 C CNN
@@
 Bat: 3*4.2V\nMon: 3.1V
 $Comp
-L +3V3 #PWR107
+L +3V3 #PWR015
 U 1 1 559CAD6D
 P 1900 4500
-F 0 "#PWR107" H 1900 4350 50  0001 C CNN
+F 0 "#PWR015" H 1900 4350 50  0001 C CNN
 F 1 "+3V3" H 1900 4640 50  0000 C CNN
 F 2 "" H 1900 4500 60  0000 C CNN
@@
 $EndComp
 $Comp
-L GND #PWR112
+L GND #PWR016
 U 1 1 559E749A
 P 10375 5850
-F 0 "#PWR112" H 10375 5600 50  0001 C CNN
+F 0 "#PWR016" H 10375 5600 50  0001 C CNN
 F 1 "GND" H 10375 5700 50  0001 C CNN
 F 2 "" H 10375 5850 60  0000 C CNN
@@
 $EndComp
 $Comp
-L GND #PWR103
+L GND #PWR017
 U 1 1 55A1A3D6
 P 5425 1400
-F 0 "#PWR103" H 5425 1150 50  0001 C CNN
+F 0 "#PWR017" H 5425 1150 50  0001 C CNN
 F 1 "GND" H 5425 1250 50  0000 C CNN
 F 2 "" H 5425 1400 60  0000 C CNN
@@
 $EndComp
 $Comp
-L +BATT #PWR102
+L +BATT #PWR018
 U 1 1 55A1ACA2
 P 5425 1200
-F 0 "#PWR102" H 5425 1050 50  0001 C CNN
+F 0 "#PWR018" H 5425 1050 50  0001 C CNN
 F 1 "+BATT" H 5425 1340 50  0000 C CNN
 F 2 "" H 5425 1200 60  0000 C CNN
@@
 $EndComp
 $Comp
-L +BATT #PWR116
+L +BATT #PWR019
 U 1 1 55A85387
 P 5550 6400
-F 0 "#PWR116" H 5550 6250 50  0001 C CNN
+F 0 "#PWR019" H 5550 6250 50  0001 C CNN
 F 1 "+BATT" H 5550 6540 50  0000 C CNN
 F 2 "" H 5550 6400 60  0000 C CNN
@@
 F 0 "P107" H 2725 2600 50  0000 C CNN
 F 1 "ARM_LED" H 2650 2900 50  0000 C CNN
-F 2 "common:JST-PA-2" H 2750 2750 60  0001 C CNN
+F 2 "ignition:JST-PA-2-VERT" H 2750 2750 60  0001 C CNN
 F 3 "" H 2750 2750 60  0000 C CNN
-F 4 "1830747" H 2750 2750 60  0001 C CNN "Farnell"
+F 4 "1830734" H 2750 2750 60  0001 C CNN "Farnell"
 	1    2750 2750
 	1    0    0    1
