File: OkGo 2/ignition/firing.sch (KiCad schematic (older format))
At the start: 75 parts, among them K201 16A SPST, K202 16A SPST, K203 16A SPST, K204 16A SPST, K205 16A SPST, P201 CH3_LED, P202 CH3_LED, P203 CH3, P204 CH1_LED, P205 CH1_LED, P206 CH1, P207 CH4_LED, P208 CH4_LED, P209 CH4, P210 CH2_LED, P211 CH2_LED, P212 CH2, Q201 BSS138BK, Q202 BSS138BK, Q203 BSS138BK, Q204 BSS138BK, Q205 BSS138BK, U201 BEZEL, U202 BEZEL, U203 BEZEL, U204 BEZEL

Commit message: ignition; first attempt at placement
Parts:
- P201, P204, P207, P210: footprint common:JST-PA-2 -> ignition:JST-PA-2-VERT; Farnell 1830747 -> 1830734
Changed lines of the file:
@@
 $EndDescr
 $Comp
-L +BATT #PWR201
+L +BATT #PWR020
 U 1 1 559E24C4
 P 2650 750
-F 0 "#PWR201" H 2650 600 50  0001 C CNN
+F 0 "#PWR020" H 2650 600 50  0001 C CNN
 F 1 "+BATT" H 2650 890 50  0000 C CNN
 F 2 "" H 2650 750 60  0000 C CNN
@@
 $EndComp
 $Comp
-L GND #PWR203
+L GND #PWR021
 U 1 1 559E24DB
 P 2650 1550
-F 0 "#PWR203" H 2650 1300 50  0001 C CNN
+F 0 "#PWR021" H 2650 1300 50  0001 C CNN
 F 1 "GND" H 2650 1400 50  0000 C CNN
 F 2 "" H 2650 1550 60  0000 C CNN
@@
 $EndComp
 $Comp
-L GND #PWR204
+L GND #PWR022
 U 1 1 559E24E8
 P 2000 1700
-F 0 "#PWR204" H 2000 1450 50  0001 C CNN
+F 0 "#PWR022" H 2000 1450 50  0001 C CNN
 F 1 "GND" H 2000 1550 50  0000 C CNN
 F 2 "" H 2000 1700 60  0000 C CNN
@@
 $EndComp
 $Comp
-L GND #PWR206
+L GND #PWR023
 U 1 1 559E250A
 P 4200 2100
-F 0 "#PWR206" H 4200 1850 50  0001 C CNN
+F 0 "#PWR023" H 4200 1850 50  0001 C CNN
 F 1 "GND" H 4200 1950 50  0000 C CNN
 F 2 "" H 4200 2100 60  0000 C CNN
@@
 $EndComp
 $Comp
-L +3V3 #PWR202
+L +3V3 #PWR024
 U 1 1 559E2520
 P 4750 1250
-F 0 "#PWR202" H 4750 1100 50  0001 C CNN
+F 0 "#PWR024" H 4750 1100 50  0001 C CNN
 F 1 "+3V3" H 4750 1390 50  0000 C CNN
 F 2 "" H 4750 1250 60  0000 C CNN
@@
 $EndComp
 $Comp
-L GND #PWR217
+L GND #PWR025
 U 1 1 559E5DCB
 P 3800 4100
-F 0 "#PWR217" H 3800 3850 50  0001 C CNN
+F 0 "#PWR025" H 3800 3850 50  0001 C CNN
 F 1 "GND" H 3800 3950 50  0000 C CNN
 F 2 "" H 3800 4100 60  0000 C CNN
@@
 $EndComp
 $Comp
-L +BATT #PWR216
+L +BATT #PWR026
 U 1 1 559E5DD9
 P 2000 3650
-F 0 "#PWR216" H 2000 3500 50  0001 C CNN
+F 0 "#PWR026" H 2000 3500 50  0001 C CNN
 F 1 "+BATT" H 2000 3790 50  0000 C CNN
 F 2 "" H 2000 3650 60  0000 C CNN
@@
 $EndComp
 $Comp
-L GND #PWR218
+L GND #PWR027
 U 1 1 559E5DF0
 P 2100 4450
-F 0 "#PWR218" H 2100 4200 50  0001 C CNN
+F 0 "#PWR027" H 2100 4200 50  0001 C CNN
 F 1 "GND" H 2100 4300 50  0000 C CNN
 F 2 "" H 2100 4450 60  0000 C CNN
@@
 $EndComp
 $Comp
-L GND #PWR220
+L GND #PWR028
 U 1 1 559E5DFD
 P 1450 4600
-F 0 "#PWR220" H 1450 4350 50  0001 C CNN
+F 0 "#PWR028" H 1450 4350 50  0001 C CNN
 F 1 "GND" H 1450 4450 50  0000 C CNN
 F 2 "" H 1450 4600 60  0000 C CNN
@@
 $EndComp
 $Comp
-L +3V3 #PWR213
+L +3V3 #PWR029
 U 1 1 559E5E03
 P 3200 3350
-F 0 "#PWR213" H 3200 3200 50  0001 C CNN
+F 0 "#PWR029" H 3200 3200 50  0001 C CNN
 F 1 "+3V3" H 3200 3490 50  0000 C CNN
 F 2 "" H 3200 3350 60  0000 C CNN
@@
 $EndComp
 $Comp
-L +3V3 #PWR214
+L +3V3 #PWR030
 U 1 1 559E5E17
 P 4250 3350
-F 0 "#PWR214" H 4250 3200 50  0001 C CNN
+F 0 "#PWR030" H 4250 3200 50  0001 C CNN
 F 1 "+3V3" H 4250 3490 50  0000 C CNN
 F 2 "" H 4250 3350 60  0000 C CNN
@@
 $EndComp
 $Comp
-L +BATT #PWR230
+L +BATT #PWR031
 U 1 1 559E5E32
 P 2050 6450
-F 0 "#PWR230" H 2050 6300 50  0001 C CNN
+F 0 "#PWR031" H 2050 6300 50  0001 C CNN
 F 1 "+BATT" H 2050 6590 50  0000 C CNN
 F 2 "" H 2050 6450 60  0000 C CNN
@@
 $EndComp
 $Comp
-L GND #PWR232
+L GND #PWR032
 U 1 1 559E5E49
 P 2150 7250
-F 0 "#PWR232" H 2150 7000 50  0001 C CNN
+F 0 "#PWR032" H 2150 7000 50  0001 C CNN
 F 1 "GND" H 2150 7100 50  0000 C CNN
 F 2 "" H 2150 7250 60  0000 C CNN
@@
 $EndComp
 $Comp
-L GND #PWR233
+L GND #PWR033
 U 1 1 559E5E56
 P 1500 7400
-F 0 "#PWR233" H 1500 7150 50  0001 C CNN
+F 0 "#PWR033" H 1500 7150 50  0001 C CNN
 F 1 "GND" H 1500 7250 50  0000 C CNN
 F 2 "" H 1500 7400 60  0000 C CNN
@@
 $EndComp
 $Comp
-L +3V3 #PWR227
+L +3V3 #PWR034
 U 1 1 559E5E5C
 P 3250 6150
-F 0 "#PWR227" H 3250 6000 50  0001 C CNN
+F 0 "#PWR034" H 3250 6000 50  0001 C CNN
 F 1 "+3V3" H 3250 6290 50  0000 C CNN
 F 2 "" H 3250 6150 60  0000 C CNN
@@
 $EndComp
 $Comp
-L +3V3 #PWR228
+L +3V3 #PWR035
 U 1 1 559E5E70
 P 4300 6150
-F 0 "#PWR228" H 4300 6000 50  0001 C CNN
+F 0 "#PWR035" H 4300 6000 50  0001 C CNN
 F 1 "+3V3" H 4300 6290 50  0000 C CNN
 F 2 "" H 4300 6150 60  0000 C CNN
@@
 $EndComp
 $Comp
-L +BATT #PWR209
+L +BATT #PWR036
 U 1 1 559E5E8B
 P 8050 2350
-F 0 "#PWR209" H 8050 2200 50  0001 C CNN
+F 0 "#PWR036" H 8050 2200 50  0001 C CNN
 F 1 "+BATT" H 8050 2490 50  0000 C CNN
 F 2 "" H 8050 2350 60  0000 C CNN
@@
 $EndComp
 $Comp
-L GND #PWR212
+L GND #PWR037
 U 1 1 559E5EA2
 P 8150 3200
-F 0 "#PWR212" H 8150 2950 50  0001 C CNN
+F 0 "#PWR037" H 8150 2950 50  0001 C CNN
 F 1 "GND" H 8150 3050 50  0000 C CNN
 F 2 "" H 8150 3200 60  0000 C CNN
@@
 $EndComp
 $Comp
-L GND #PWR215
+L GND #PWR038
 U 1 1 559E5EAF
 P 7500 3350
-F 0 "#PWR215" H 7500 3100 50  0001 C CNN
+F 0 "#PWR038" H 7500 3100 50  0001 C CNN
 F 1 "GND" H 7500 3200 50  0000 C CNN
 F 2 "" H 7500 3350 60  0000 C CNN
@@
 $EndComp
 $Comp
-L +3V3 #PWR207
+L +3V3 #PWR039
 U 1 1 559E5EB5
 P 9250 2100
-F 0 "#PWR207" H 9250 1950 50  0001 C CNN
+F 0 "#PWR039" H 9250 1950 50  0001 C CNN
 F 1 "+3V3" H 9250 2240 50  0000 C CNN
 F 2 "" H 9250 2100 60  0000 C CNN
@@
 $EndComp
 $Comp
-L +3V3 #PWR208
+L +3V3 #PWR040
 U 1 1 559E5EC9
 P 10300 2100
-F 0 "#PWR208" H 10300 1950 50  0001 C CNN
+F 0 "#PWR040" H 10300 1950 50  0001 C CNN
 F 1 "+3V3" H 10300 2240 50  0000 C CNN
 F 2 "" H 10300 2100 60  0000 C CNN
@@
 $EndComp
 $Comp
-L +BATT #PWR223
+L +BATT #PWR041
 U 1 1 559E5EE4
 P 8050 5225
-F 0 "#PWR223" H 8050 5075 50  0001 C CNN
+F 0 "#PWR041" H 8050 5075 50  0001 C CNN
 F 1 "+BATT" H 8050 5365 50  0000 C CNN
 F 2 "" H 8050 5225 60  0000 C CNN
@@
 $EndComp
 $Comp
-L GND #PWR226
+L GND #PWR042
 U 1 1 559E5EFB
 P 8150 6050
-F 0 "#PWR226" H 8150 5800 50  0001 C CNN
+F 0 "#PWR042" H 8150 5800 50  0001 C CNN
 F 1 "GND" H 8150 5900 50  0000 C CNN
 F 2 "" H 8150 6050 60  0000 C CNN
@@
 $EndComp
 $Comp
-L GND #PWR229
+L GND #PWR043
 U 1 1 559E5F08
 P 7450 6200
-F 0 "#PWR229" H 7450 5950 50  0001 C CNN
+F 0 "#PWR043" H 7450 5950 50  0001 C CNN
 F 1 "GND" H 7450 6050 50  0000 C CNN
 F 2 "" H 7450 6200 60  0000 C CNN
@@
 $EndComp
 $Comp
-L +3V3 #PWR221
+L +3V3 #PWR044
 U 1 1 559E5F0E
 P 9250 4950
-F 0 "#PWR221" H 9250 4800 50  0001 C CNN
+F 0 "#PWR044" H 9250 4800 50  0001 C CNN
 F 1 "+3V3" H 9250 5090 50  0000 C CNN
 F 2 "" H 9250 4950 60  0000 C CNN
@@
 $EndComp
 $Comp
-L +3V3 #PWR222
+L +3V3 #PWR045
 U 1 1 559E5F22
 P 10300 4950
-F 0 "#PWR222" H 10300 4800 50  0001 C CNN
+F 0 "#PWR045" H 10300 4800 50  0001 C CNN
 F 1 "+3V3" H 10300 5090 50  0000 C CNN
 F 2 "" H 10300 4950 60  0000 C CNN
@@
 F 0 "P204" H 1025 3050 50  0000 C CNN
 F 1 "CH1_LED" H 950 3350 50  0000 C CNN
-F 2 "common:JST-PA-2" H 1050 3200 60  0001 C CNN
+F 2 "ignition:JST-PA-2-VERT" H 1050 3200 60  0001 C CNN
 F 3 "" H 1050 3200 60  0000 C CNN
-F 4 "1830747" H 1050 3200 60  0001 C CNN "Farnell"
+F 4 "1830734" H 1050 3200 60  0001 C CNN "Farnell"
 	1    1050 3200
 	1    0    0    1
@@
 $EndComp
 $Comp
-L GND #PWR231
+L GND #PWR046
 U 1 1 55A99294
 P 3850 6900
-F 0 "#PWR231" H 3850 6650 50  0001 C CNN
+F 0 "#PWR046" H 3850 6650 50  0001 C CNN
 F 1 "GND" H 3850 6750 50  0000 C CNN
 F 2 "" H 3850 6900 60  0000 C CNN
@@
 F 0 "P210" H 1050 5850 50  0000 C CNN
 F 1 "CH2_LED" H 1000 6150 50  0000 C CNN
-F 2 "common:JST-PA-2" H 1100 6000 60  0001 C CNN
+F 2 "ignition:JST-PA-2-VERT" H 1100 6000 60  0001 C CNN
 F 3 "" H 1100 6000 60  0000 C CNN
-F 4 "1830747" H 1100 6000 60  0001 C CNN "Farnell"
+F 4 "1830734" H 1100 6000 60  0001 C CNN "Farnell"
 	1    1100 6000
 	1    0    0    1
@@
 $EndComp
 $Comp
-L GND #PWR211
+L GND #PWR047
 U 1 1 55A9A2B3
 P 9850 2850
-F 0 "#PWR211" H 9850 2600 50  0001 C CNN
+F 0 "#PWR047" H 9850 2600 50  0001 C CNN
 F 1 "GND" H 9850 2700 50  0000 C CNN
 F 2 "" H 9850 2850 60  0000 C CNN
@@
 F 0 "P201" H 6775 1950 50  0000 C CNN
 F 1 "CH3_LED" H 6700 2250 50  0000 C CNN
-F 2 "common:JST-PA-2" H 6800 2100 60  0001 C CNN
+F 2 "ignition:JST-PA-2-VERT" H 6800 2100 60  0001 C CNN
 F 3 "" H 6800 2100 60  0000 C CNN
-F 4 "1830747" H 6800 2100 60  0001 C CNN "Farnell"
+F 4 "1830734" H 6800 2100 60  0001 C CNN "Farnell"
 	1    6800 2100
 	1    0    0    1
@@
 $EndComp
 $Comp
-L GND #PWR225
+L GND #PWR048
 U 1 1 55A9B178
 P 9850 5700
-F 0 "#PWR225" H 9850 5450 50  0001 C CNN
+F 0 "#PWR048" H 9850 5450 50  0001 C CNN
 F 1 "GND" H 9850 5550 50  0000 C CNN
 F 2 "" H 9850 5700 60  0000 C CNN
@@
 F 0 "P207" H 6775 4750 50  0000 C CNN
 F 1 "CH4_LED" H 6700 5050 50  0000 C CNN
-F 2 "common:JST-PA-2" H 6800 4900 60  0001 C CNN
+F 2 "ignition:JST-PA-2-VERT" H 6800 4900 60  0001 C CNN
 F 3 "" H 6800 4900 60  0000 C CNN
-F 4 "1830747" H 6800 4900 60  0001 C CNN "Farnell"
+F 4 "1830734" H 6800 4900 60  0001 C CNN "Farnell"
 	1    6800 4900
 	1    0    0    1
@@
 $EndComp
 $Comp
-L +BATT #PWR219
+L +BATT #PWR049
 U 1 1 55AAA64D
 P 6500 4550
-F 0 "#PWR219" H 6500 4400 50  0001 C CNN
+F 0 "#PWR049" H 6500 4400 50  0001 C CNN
 F 1 "+BATT" H 6500 4690 50  0000 C CNN
 F 2 "" H 6500 4550 60  0000 C CNN
@@
 	8200 2250 8200 2400
 $Comp
-L +BATT #PWR205
+L +BATT #PWR050
 U 1 1 55AB4F23
 P 6450 1750
-F 0 "#PWR205" H 6450 1600 50  0001 C CNN
+F 0 "#PWR050" H 6450 1600 50  0001 C CNN
 F 1 "+BATT" H 6450 1890 50  0000 C CNN
 F 2 "" H 6450 1750 60  0000 C CNN
@@
 	6200 500  6200 7800
 $Comp
-L +BATT #PWR210
+L +BATT #PWR051
 U 1 1 55AB71ED
 P 700 2850
-F 0 "#PWR210" H 700 2700 50  0001 C CNN
+F 0 "#PWR051" H 700 2700 50  0001 C CNN
 F 1 "+BATT" H 700 2990 50  0000 C CNN
 F 2 "" H 700 2850 60  0000 C CNN
@@
 	750  5950 900  5950
 $Comp
-L +BATT #PWR224
+L +BATT #PWR052
 U 1 1 55ABA6A0
 P 750 5650
-F 0 "#PWR224" H 750 5500 50  0001 C CNN
+F 0 "#PWR052" H 750 5500 50  0001 C CNN
 F 1 "+BATT" H 750 5790 50  0000 C CNN
 F 2 "" H 750 5650 60  0000 C CNN

Commit message: ignition test routing somewhat done
Connections:
- net +BATT: now also D217.1 (K); no longer D217.2 (A)
- net at K205.1, P210.1 (P1), Q205.3 (D): now also D217.2 (A); no longer D217.1 (K)
Changed lines of the file:
@@
 U 1 1 55AA9E3E
 P 1950 6600
-F 0 "D217" H 1900 6680 50  0000 L CNN
+F 0 "D217" H 1850 6500 50  0000 L CNN
 F 1 "MBR2H200SFT1G" H 1670 6520 50  0001 L CNN
 F 2 "ignition:SOD-123FL" V 1950 6600 60  0001 C CNN
@@
 F 4 "2452032" H 1950 6600 60  0001 C CNN "Farnell"
 	1    1950 6600
-	0    -1   -1   0
+	0    1    1    0
 $EndComp
 Connection ~ 1950 6700
