File: OkGo 2/ignition/firing.sch (KiCad schematic (older format))
At the start: 75 parts, among them K201 16A SPST, K202 16A SPST, K203 16A SPST, K204 16A SPST, K205 16A SPST, P201 CH3_LED, P202 CH3_LED, P203 CH3, P204 CH1_LED, P205 CH1_LED, P206 CH1, P207 CH4_LED, P208 CH4_LED, P209 CH4, P210 CH2_LED, P211 CH2_LED, P212 CH2, Q201 BSS138BK, Q202 BSS138BK, Q203 BSS138BK, Q204 BSS138BK, Q205 BSS138BK, U201 BEZEL, U202 BEZEL, U203 BEZEL, U204 BEZEL

Commit message: BOM updates
Parts:
- D203: Farnell 1855546 -> 2293491
- R205, R215: value 430 -> 470R; Farnell (none) -> 2332067
- R209: value 510R -> 470R; Farnell (none) -> 2332067
- R219: value 510 -> 470R; Farnell (none) -> 2332067
Changed lines of the file:
@@
 P 700 3000
 F 0 "R209" V 600 2900 50  0000 C CNN
-F 1 "510R" V 700 3000 50  0000 C CNN
+F 1 "470R" V 700 3000 50  0000 C CNN
 F 2 "Resistors_SMD:R_0805" V 630 3000 30  0001 C CNN
 F 3 "" H 700 3000 30  0000 C CNN
+F 4 "2332067" H 700 3000 60  0001 C CNN "Farnell"
 	1    700  3000
 	-1   0    0    1
@@
 P 750 5800
 F 0 "R219" V 650 5700 50  0000 C CNN
-F 1 "510" V 750 5800 50  0000 C CNN
+F 1 "470R" V 750 5800 50  0000 C CNN
 F 2 "Resistors_SMD:R_0805" V 680 5800 30  0001 C CNN
 F 3 "" H 750 5800 30  0000 C CNN
+F 4 "2332067" H 750 5800 60  0001 C CNN "Farnell"
 	1    750  5800
 	-1   0    0    1
@@
 P 6450 1900
 F 0 "R205" V 6350 1800 50  0000 C CNN
-F 1 "430" V 6450 1900 50  0000 C CNN
+F 1 "470R" V 6450 1900 50  0000 C CNN
 F 2 "Resistors_SMD:R_0805" V 6380 1900 30  0001 C CNN
 F 3 "" H 6450 1900 30  0000 C CNN
+F 4 "2332067" H 6450 1900 60  0001 C CNN "Farnell"
 	1    6450 1900
 	-1   0    0    1
@@
 F 2 "" H 7350 2050 60  0000 C CNN
 F 3 "" H 7350 2050 60  0000 C CNN
-F 4 "1855546" H 7350 2050 60  0001 C CNN "Farnell"
+F 4 "2293491" H 7350 2050 60  0001 C CNN "Farnell"
 	1    7350 2050
 	-1   0    0    1
@@
 P 6500 4700
 F 0 "R215" V 6400 4600 50  0000 C CNN
-F 1 "430" V 6500 4700 50  0000 C CNN
+F 1 "470R" V 6500 4700 50  0000 C CNN
 F 2 "Resistors_SMD:R_0805" V 6430 4700 30  0001 C CNN
 F 3 "" H 6500 4700 30  0000 C CNN
+F 4 "2332067" H 6500 4700 60  0001 C CNN "Farnell"
 	1    6500 4700
 	-1   0    0    1
