File: okgo2mini/board/okgo2mini.kicad_pcb (KiCad board)
At the start: 2 copper layers, 43 parts, among them IC1 BQ24232HA, IC2 STM32F051K6T7, IC3 ADP3335, IC4 TPS62130, J1 BATT, J2 MICROUSB STRAIGHT, J3 PYRO, P1 SWD, P2 SWD_TC, P3 ANT, SW1 SWITCH_SPST, U1 RFM95W

Commit message: WIP
Parts:
- added REF**: M3_MOUNT, agg:M3_MOUNT, F.Cu at (165.0, 135.0)
- added REF**: M3_MOUNT, agg:M3_MOUNT, F.Cu at (205.0, 135.0)
- added REF**: M3_MOUNT, agg:M3_MOUNT, F.Cu at (205.0, 95.0)
- added REF**: M3_MOUNT, agg:M3_MOUNT, F.Cu at (165.0, 95.0)
- SW1: footprint okgo2mini:710xxxxV3xx -> okgo2mini:120x-M1-xx-C; moved to B.Cu
- moved P3 83.0 mm to (207.0, 105.5), turned to 270 degrees
- moved U1 82.3 mm to (192.5, 98.5)
- moved J2 80.3 mm to (185.0, 110.8)
- moved D5 78.5 mm to (173.2, 126.8), turned to 90 degrees
- moved C12 74.9 mm to (119.7, 115.5), turned to 90 degrees
- moved SW1 74.6 mm to (176.0, 98.0), turned to 90 degrees
- moved D4 74.0 mm to (202.8, 104.8), turned to 90 degrees
- moved P2 73.1 mm to (204.0, 125.8)
- moved C9 72.4 mm to (178.8, 115.5), turned to 90 degrees
- moved C11 70.5 mm to (118.2, 115.5), turned to 90 degrees
- moved P1 70.2 mm to (204.5, 117.8), turned to 90 degrees
- moved IC4 68.9 mm to (124.0, 115.8), turned to 180 degrees
- moved IC2 66.4 mm to (194.8, 117.8)
- moved J3 66.0 mm to (168.6, 126.8), turned to 90 degrees
- moved C17 65.2 mm to (125.5, 120.0), turned to 180 degrees
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Routing:
- net /PYRO_POWER: track 0.00 -> 4.56 mm
- net GND: track 0.00 -> 3.43 mm
- net Net-(IC1-Pad16): track 0.00 -> 1.64 mm
- added copper zone on F.Cu, net +3V3
- added copper zone on F.Cu, net +5V
- added copper zone on F.Cu, net /PYRO_POWER
- added copper zone on F.Cu, net /VBAT
- added copper zone on B.Cu, net GND
- added copper zone on F.Cu, net Net-(IC4-Pad1)
Other:
- board outline added: 50 x 50 mm
- rule pad_to_mask_clearance: 0.2 -> 0

Commit message: WIP
Parts:
- removed REF** (x4): M3_MOUNT, agg:M3_MOUNT
- added P4: u.FL, unchecked:uFL-R-SMT, F.Cu at (202.4, 105.5)
- added Q1: Si5515CDC, agg:ChipFET-1206-8, F.Cu at (181.4, 133.1)
- added R8: 100k, agg:0603, F.Cu at (181.2, 130.2)
- added R9: 100k, agg:0603, F.Cu at (177.2, 133.9)
- added X1: M3 Mount, agg:M3_MOUNT, F.Cu at (165.0, 135.0)
- added X2: M3 Mount, agg:M3_MOUNT, F.Cu at (165.0, 95.0)
- added X3: M3 Mount, agg:M3_MOUNT, F.Cu at (205.0, 95.0)
- added X4: M3 Mount, agg:M3_MOUNT, F.Cu at (205.0, 135.0)
- D1, D2: footprint agg:0805-LED -> LEDs:LED_D3.0mm
- P3: value ANT -> SMA
- SW1: value SWITCH_SPST -> SWITCH_DPDT
- moved D6 115.7 mm to (187.4, 128.4), turned to 180 degrees
- moved D3 110.3 mm to (183.4, 128.4)
- moved R7 91.7 mm to (186.2, 133.3), turned to 270 degrees
- moved R6 90.7 mm to (184.7, 133.3), turned to 90 degrees
- moved C11 49.9 mm to (166.2, 129.1)
- moved C12 49.9 mm to (167.7, 129.1)
- moved C13 49.9 mm to (169.2, 128.0)
- moved IC4 49.9 mm to (172.0, 129.3)
- moved L1 49.9 mm to (177.3, 130.8)
- moved C17 49.5 mm to (173.2, 133.1), turned to 270 degrees
- moved C16 48.5 mm to (171.7, 133.1), turned to 270 degrees
- moved C1 34.3 mm to (171.2, 123.0), turned to 270 degrees
- moved C6 34.1 mm to (168.9, 124.5), turned to 0 degrees
- moved R1 29.2 mm to (171.2, 119.8), turned to 270 degrees
- moved IC1 28.0 mm to (168.1, 121.4), turned to 270 degrees
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Connections:
- net /FIRE renamed /FIRE1
- D5 pad 1: Net-(C16-Pad1) -> Net-(D5-Pad1)
- J2 pad 1: +5V -> Net-(J2-Pad1)
- J3 pad 2: Net-(C16-Pad1) -> Net-(D5-Pad1)
- R6 pad 1: Net-(C16-Pad1) -> Net-(D5-Pad1)
- R7 pad 2: Net-(C16-Pad1) -> Net-(D5-Pad1)
- SW1 pad 3: (no net) -> Net-(SW1-Pad3)
- SW1 pad 4: (no net) -> +5V
- SW1 pad 5: (no net) -> Net-(J2-Pad1)
- SW1 pad 6: (no net) -> Net-(SW1-Pad6)
Routing:
- net GND: track 3.43 -> 49.6 mm, vias 0 -> 5
- net /BATT_TEMP: track 0.00 -> 27.6 mm
- net Net-(D5-Pad1): track 0.00 -> 16.8 mm
- net Net-(J1-Pad1): track 0.00 -> 14.4 mm
- net /PYRO_POWER: track 4.56 -> 15.9 mm
- net Net-(J2-Pad1): track 0.00 -> 11.2 mm
- net Net-(D4-Pad1): track 0.00 -> 10.0 mm
- net +5V: track 0.07 -> 8.62 mm
- net Net-(C16-Pad1): track 0.00 -> 7.35 mm
- net Net-(Q1-Pad4): track 0.00 -> 6.79 mm
- net +3V3: track 0.00 -> 5.89 mm
- net /VBAT: track 0.00 -> 5.74 mm
- net /CONT: track 0.00 -> 4.10 mm
- net /CONT_EN: track 0.00 -> 4.10 mm
- net Net-(IC4-Pad1): track 0.00 -> 3.86 mm
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- removed copper zone on F.Cu, net +3V3
